Commit message: corrected mass for one wheel with different value

File: src/my_robot/urdf/my_robot.xacro (robot description, xacro)
@@ -160,5 +160,5 @@
     </visual>
     <inertial>
-      <mass value="5.0"/>
+      <mass value="10.0"/>
       <origin xyz="0.0 0 0" rpy=" 0 0 0"/>
       <inertia

Commit message: modify robot to locate radar in a lower possition able to read tables collisions

File: src/my_robot/urdf/my_robot.xacro (robot description, xacro)
@@ -22,5 +22,5 @@
       <origin xyz="0 0 0" rpy=" 0 0 0"/>
       <geometry>
-        <box size=".4 .2 .1"/>
+        <box size="0.6 0.2 0.04"/>
       </geometry>
     </collision>
@@ -28,17 +28,17 @@
       <origin xyz="0 0 0" rpy=" 0 0 0"/>
       <geometry>
-        <box size=".6 .2 .1"/>
+        <box size="0.6 0.2 0.04"/>
       </geometry>
     </visual>
     <collision name='chassis_top_collision'>
-      <origin xyz="0 0 0.075" rpy=" 0 0 0"/>
-      <geometry>
-        <box size=".05 .05 .05"/>
+      <origin xyz="0 0 0.065" rpy=" 0 0 0"/>
+      <geometry>
+        <box size="0.25 0.05 0.09"/>
       </geometry>
     </collision>
     <visual name='chassis_top_visual'>
-      <origin xyz="0 0 0.075" rpy=" 0 0 0"/>
-      <geometry>
-        <box size=".05 .05 .05"/>
+      <origin xyz="0 0 0.065" rpy=" 0 0 0"/>
+      <geometry>
+        <box size="0.25 0.05 0.09"/>
       </geometry>
     </visual>
@@ -171,5 +171,5 @@
 	<!-- sensors -->
   <joint type="fixed" name="camera_joint">
-    <origin xyz="0.325 0 0" rpy="0 0 0"/>
+    <origin xyz="0.275 0 0.045" rpy="0 0 0"/>
     <child link="camera"/>
     <parent link="chassis"/>
@@ -200,5 +200,5 @@
 	</link>
   <joint type="fixed" name="hokuyo_joint">
-    <origin xyz="-0.26 0 0.205" rpy="0 0 0"/>
+    <origin xyz="0.275 0 -0.055" rpy="0 0 0"/>
     <child link="hokuyo"/>
     <parent link="chassis"/>
@@ -213,5 +213,5 @@
     </collision>
     <visual name='hokuyo_visual'>
-      <origin xyz="0 0 0" rpy=" 0 0 0"/>
+      <origin xyz="0 0 0" rpy=" 3.14159 0 0"/>
       <geometry>
 				<mesh filename="package://my_robot/meshes/hokuyo.dae" />
@@ -230,5 +230,5 @@
 	<!-- plate -->
   <joint type="fixed" name="plate_hinge">
-    <origin xyz="0 0 0.11" rpy="0 0 0"/>
+    <origin xyz="0 0 0.12" rpy="0 0 0"/>
     <child link="plate"/>
     <parent link="chassis"/>
@@ -257,16 +257,4 @@
       />
     </inertial>
-    <collision name='plate_top_collision'>
-      <origin xyz="-0.26 0 0.035" rpy=" 0 0 0"/>
-      <geometry>
-        <box size=".07 .07 .05"/>
-      </geometry>
-    </collision>
-    <visual name='plate_top_visual'>
-      <origin xyz="-0.26 0 0.035" rpy=" 0 0 0"/>
-      <geometry>
-        <box size=".07 .07 .05"/>
-      </geometry>
-    </visual>
 	</link>
 </robot>

Commit message: incorporated diff move controller for the robot to move better in the path planner

File: src/my_robot/urdf/my_robot.xacro (robot description, xacro)
@@ -1,4 +1,4 @@
 <?xml version='1.0'?>
-<robot name="my_robot" xmlns:xacro="http://www.ros.org/wiki/xacro">
+<robot name="my_robot" xmlns:xacro="http://ros.org/wiki/xacro">
 	<xacro:include filename="$(find my_robot)/urdf/my_robot.gazebo"/>
   <link name="robot_footprint"></link>
@@ -53,4 +53,14 @@
     <dynamics damping="1.0" friction="1.0"/>
   </joint>
+  <transmission name="left_front_wheel_trans">
+    <type>transmission_interface/SimpleTransmission</type>
+    <joint name="left_front_wheel_hinge">
+      <hardwareInterface>hardware_interface/EffortJointInterface</hardwareInterface>
+		</joint>
+    <actuator name="left_front_wheel_actuator">
+      <hardwareInterface>EffortJointInterface</hardwareInterface>
+      <mechanicalReduction>1</mechanicalReduction>
+      </actuator>
+  </transmission>
 	<link name='left_front_wheel'>
     <collision name='left_front_wheel_collision'>
@@ -84,4 +94,14 @@
     <dynamics damping="1.0" friction="1.0"/>
   </joint>
+  <transmission name="right_front_wheel_trans">
+    <type>transmission_interface/SimpleTransmission</type>
+    <joint name="right_front_wheel_hinge">
+      <hardwareInterface>hardware_interface/EffortJointInterface</hardwareInterface>
+		</joint>
+    <actuator name="right_front_wheel_actuator">
+      <hardwareInterface>EffortJointInterface</hardwareInterface>
+      <mechanicalReduction>1</mechanicalReduction>
+      </actuator>
+  </transmission>
 	<link name='right_front_wheel'>
     <collision name='right_front_wheel_collision'>
@@ -115,4 +135,14 @@
     <dynamics damping="1.0" friction="1.0"/>
   </joint>
+  <transmission name="left_back_wheel_trans">
+    <type>transmission_interface/SimpleTransmission</type>
+    <joint name="left_back_wheel_hinge">
+      <hardwareInterface>hardware_interface/EffortJointInterface</hardwareInterface>
+		</joint>
+    <actuator name="left_back_wheel_actuator">
+      <hardwareInterface>EffortJointInterface</hardwareInterface>
+      <mechanicalReduction>1</mechanicalReduction>
+      </actuator>
+  </transmission>
 	<link name='left_back_wheel'>
     <collision name='left_back_wheel_collision'>
@@ -146,4 +176,14 @@
     <dynamics damping="1.0" friction="1.0"/>
   </joint>
+  <transmission name="right_back_wheel_trans">
+    <type>transmission_interface/SimpleTransmission</type>
+    <joint name="right_back_wheel_hinge">
+      <hardwareInterface>hardware_interface/EffortJointInterface</hardwareInterface>
+		</joint>
+    <actuator name="right_back_wheel_actuator">
+      <hardwareInterface>EffortJointInterface</hardwareInterface>
+      <mechanicalReduction>1</mechanicalReduction>
+      </actuator>
+  </transmission>
 	<link name='right_back_wheel'>
     <collision name='right_back_wheel_collision'>

Commit message: last modifications for project submission

File: src/my_robot/urdf/my_robot.xacro (robot description, xacro)
@@ -73,5 +73,5 @@
       <origin xyz="0 -0.02 0" rpy=" 0 1.5707 0"/>
       <geometry>
-				<mesh filename="package://my_robot/meshes/mecanum0.stl" scale="1 1 1"/>
+				<mesh filename="package://my_robot/meshes/mecanum.dae" scale="1 1 1"/>
       </geometry>
     </visual>
